File: schematics/stingray.kicad_pcb (KiCad board)
At the start: 2 copper layers, 77 x 54.6 mm, 15 parts, among them J1 Target Board, K1 G6RL-1, P8 BeagleBone_Black_Header, P9 BeagleBone_Black_Header, Q1 MPSA29

Commit message: PCB rev A2
Parts:
- D1: footprint Diode_THT:D_DO-41_SOD81_P7.62mm_Horizontal -> Diode_THT:D_DO-41_SOD81_P10.16mm_Horizontal
- Q1: footprint Package_TO_SOT_THT:TO-92_Inline_Wide -> Package_TO_SOT_THT:TO-92_Inline
- R1, R2, R3: footprint Resistor_THT:R_Axial_DIN0207_L6.3mm_D2.5mm_P7.62mm_Horizontal -> Resistor_THT:R_Axial_DIN0207_L6.3mm_D2.5mm_P10.16mm_Horizontal
- moved R2 2.59 mm to (147.5, 85.7)
- moved Q1 2.02 mm to (149.3, 91.0)
- moved J1 1.39 mm to (105.6, 95.8)
- moved C2 1.00 mm to (129.0, 84.0)
Routing:
- net +5V: track 76.1 -> 78.6 mm
- net Net-(J1-Pad3): track 11.5 -> 12.9 mm
- net Net-(J1-Pad2): track 14.6 -> 16.0 mm
- net GND: track 8.12 -> 9.46 mm
- net Net-(D1-Pad2): track 28.5 -> 29.4 mm
- net GPIO_48: track 14.1 -> 13.4 mm
Other:
- board text added: "REV A2"
- board text removed: "REV A1"
