File: schematics/stingray.kicad_sch (KiCad schematic)
At the start: 15 parts, among them J1 Target Board, K1 G6RL-1, P8 BeagleBone_Black_Header, P9 BeagleBone_Black_Header, Q1 MPSA29

Commit message: Schematic cleanup
Other:
- note added: "Headers"
- note added: "Mounting"
- note added: "Target Controller"
- note removed: "SYS_5V"
- note removed: "VDD_3V3"
- moved on the sheet: C1, C2, D1, H1, H2, H3, H4, J1, K1, P8, P9, Q1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

Commit message: PCB rev A2
Parts:
- R1, R2, R3: footprint Resistor_THT:R_Axial_DIN0207_L6.3mm_D2.5mm_P7.62mm_Horizontal -> Resistor_THT:R_Axial_DIN0207_L6.3mm_D2.5mm_P10.16mm_Horizontal
Changed lines of the file:
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@@
     (title "Stingray BBB Cape")
     (date "2023-01-02")
-    (rev "A1")
+    (rev "A2")
     (company "An Alex McLain Design")
     (comment 1 "AM")
   )
+  (junction (at 83.82 40.64) (diameter 0) (color 0 0 0 0)
+  )
   (junction (at 158.75 64.77) (diameter 0) (color 0 0 0 0)
   )
@@
   )
   (junction (at 158.75 48.26) (diameter 0) (color 0 0 0 0)
-  )
-  (junction (at 83.82 40.64) (diameter 0) (color 0 0 0 0)
   )
   (junction (at 147.32 48.26) (diameter 0) (color 0 0 0 0)
@@
     (stroke (width 0) (type default) (color 0 0 0 0))
   )
+  (wire (pts (xy 130.81 64.77) (xy 130.81 45.72))
+    (stroke (width 0) (type default) (color 0 0 0 0))
+  )
+  (wire (pts (xy 50.8 134.62) (xy 50.8 148.59))
+    (stroke (width 0) (type default) (color 0 0 0 0))
+  )
+  (wire (pts (xy 74.93 96.52) (xy 104.14 96.52))
+    (stroke (width 0) (type default) (color 0 0 0 0))
+  )
+  (wire (pts (xy 104.14 40.64) (xy 104.14 46.99))
+    (stroke (width 0) (type default) (color 0 0 0 0))
+  )
+  (wire (pts (xy 105.41 140.97) (xy 105.41 148.59))
+    (stroke (width 0) (type default) (color 0 0 0 0))
+  )
+  (wire (pts (xy 114.3 43.18) (xy 172.72 43.18))
+    (stroke (width 0) (type default) (color 0 0 0 0))
+  )
+  (wire (pts (xy 198.12 40.64) (xy 198.12 43.18))
+    (stroke (width 0) (type default) (color 0 0 0 0))
+  )
   (wire (pts (xy 83.82 33.02) (xy 83.82 40.64))
-    (stroke (width 0) (type default) (color 0 0 0 0))
-  )
-  (wire (pts (xy 130.81 64.77) (xy 130.81 45.72))
-    (stroke (width 0) (type default) (color 0 0 0 0))
-  )
-  (wire (pts (xy 50.8 134.62) (xy 50.8 148.59))
-    (stroke (width 0) (type default) (color 0 0 0 0))
-  )
-  (wire (pts (xy 74.93 96.52) (xy 104.14 96.52))
-    (stroke (width 0) (type default) (color 0 0 0 0))
-  )
-  (wire (pts (xy 104.14 40.64) (xy 104.14 46.99))
-    (stroke (width 0) (type default) (color 0 0 0 0))
-  )
-  (wire (pts (xy 105.41 140.97) (xy 105.41 148.59))
-    (stroke (width 0) (type default) (color 0 0 0 0))
-  )
-  (wire (pts (xy 114.3 43.18) (xy 172.72 43.18))
-    (stroke (width 0) (type default) (color 0 0 0 0))
-  )
-  (wire (pts (xy 198.12 40.64) (xy 198.12 43.18))
     (stroke (width 0) (type default) (color 0 0 0 0))
   )
@@
       (effects (font (size 1.27 1.27)) (justify left))
     )
-    (property "Footprint" "Resistor_THT:R_Axial_DIN0207_L6.3mm_D2.5mm_P7.62mm_Horizontal" (id 2) (at 75.946 87.884 90)
+    (property "Footprint" "Resistor_THT:R_Axial_DIN0207_L6.3mm_D2.5mm_P10.16mm_Horizontal" (id 2) (at 75.946 87.884 90)
       (effects (font (size 1.27 1.27)) hide)
     )
@@
     (property "Reference" "R2" (id 0) (at 86.36 73.533 90))
     (property "Value" "1k" (id 1) (at 86.36 75.8444 90))
-    (property "Footprint" "Resistor_THT:R_Axial_DIN0207_L6.3mm_D2.5mm_P7.62mm_Horizontal" (id 2) (at 86.106 79.756 90)
+    (property "Footprint" "Resistor_THT:R_Axial_DIN0207_L6.3mm_D2.5mm_P10.16mm_Horizontal" (id 2) (at 86.106 79.756 90)
       (effects (font (size 1.27 1.27)) hide)
     )
@@
       (effects (font (size 1.27 1.27)) (justify left))
     )
-    (property "Footprint" "Resistor_THT:R_Axial_DIN0207_L6.3mm_D2.5mm_P7.62mm_Horizontal" (id 2) (at 139.446 56.134 90)
+    (property "Footprint" "Resistor_THT:R_Axial_DIN0207_L6.3mm_D2.5mm_P10.16mm_Horizontal" (id 2) (at 139.446 56.134 90)
       (effects (font (size 1.27 1.27)) hide)
     )
@@
     )
     (path "/00000000-0000-0000-0000-0000638d2382"
-      (reference "R1") (unit 1) (value "22k") (footprint "Resistor_THT:R_Axial_DIN0207_L6.3mm_D2.5mm_P7.62mm_Horizontal")
+      (reference "R1") (unit 1) (value "22k") (footprint "Resistor_THT:R_Axial_DIN0207_L6.3mm_D2.5mm_P10.16mm_Horizontal")
     )
     (path "/00000000-0000-0000-0000-0000638d2f42"
-      (reference "R2") (unit 1) (value "1k") (footprint "Resistor_THT:R_Axial_DIN0207_L6.3mm_D2.5mm_P7.62mm_Horizontal")
+      (reference "R2") (unit 1) (value "1k") (footprint "Resistor_THT:R_Axial_DIN0207_L6.3mm_D2.5mm_P10.16mm_Horizontal")
     )
     (path "/00000000-0000-0000-0000-000063b06001"
-      (reference "R3") (unit 1) (value "1M") (footprint "Resistor_THT:R_Axial_DIN0207_L6.3mm_D2.5mm_P7.62mm_Horizontal")
-    )
-  )
+      (reference "R3") (unit 1) (value "1M") (footprint "Resistor_THT:R_Axial_DIN0207_L6.3mm_D2.5mm_P10.16mm_Horizontal")
+    )
+  )
